Commit message: Fixed ODAS + FAIRINO arm movement

File: src/dracoviloc_description/urdf/dracoviloc.urdf.xacro (robot description, xacro)
@@ -41,4 +41,27 @@
             rpy="0 0 0"/>
   </joint>
+  <!-- UMA16v2 microphone-array frame. ODAS directions are expressed in this
+       frame; +Z is normal to the microphone plane. These placeholder mount
+       dimensions must be replaced with measurements from the final bracket. -->
+  <xacro:property name="odas_mount_x" value="0.0"/>
+  <xacro:property name="odas_mount_y" value="0.0"/>
+  <xacro:property name="odas_mount_z" value="0.13"/>
+  <link name="odas_link">
+    <visual>
+      <geometry><box size="0.126 0.126 0.008"/></geometry>
+      <material name="odas_blue"><color rgba="0.05 0.25 0.8 0.8"/></material>
+    </visual>
+    <collision><geometry><box size="0.126 0.126 0.008"/></geometry></collision>
+    <inertial>
+      <mass value="0.08"/>
+      <inertia ixx="0.000106" ixy="0" ixz="0"
+               iyy="0.000106" iyz="0" izz="0.000212"/>
+    </inertial>
+  </link>
+  <joint name="wrist3_to_odas" type="fixed">
+    <parent link="wrist3_link"/>
+    <child link="odas_link"/>
+    <origin xyz="${odas_mount_x} ${odas_mount_y} ${odas_mount_z}" rpy="0 0 0"/>
+  </joint>
   <ros2_control name="fairino_arm_system" type="system">
     <hardware>

Commit message: updted EKF, fixed layout of the project

File: src/dracoviloc_description/urdf/dracoviloc.urdf.xacro (robot description, xacro)
@@ -1,5 +1,4 @@
 <?xml version="1.0"?>
 <robot xmlns:xacro="http://www.ros.org/wiki/xacro" name="dracoviloc">
-  <xacro:arg name="sim" default="true"/>
   <xacro:arg name="robot_ip" default="192.168.58.2"/>
   <xacro:arg name="initial_positions_file"
@@ -7,5 +6,4 @@
   <xacro:arg name="ros2_controllers_file"
     default="$(find dracoviloc_bringup)/config/ros2_controllers.yaml"/>
-  <xacro:property name="sim" value="$(arg sim)"/>
   <xacro:property name="initial_positions"
     value="${xacro.load_yaml('$(arg initial_positions_file)')['initial_positions']}"/>
@@ -16,5 +14,5 @@
     <child link="base_link"/>
   </joint>
-  <xacro:fairino3_v6_robot_prefixed prefix="" sim="${sim}"/>
+  <xacro:fairino3_v6_robot_prefixed prefix=""/>
   <!-- D435i body convention inherited from Vicoman:
        +X forward/view direction, +Y left, +Z up.
@@ -66,11 +64,6 @@
   <ros2_control name="fairino_arm_system" type="system">
     <hardware>
-      <xacro:if value="${sim}">
-        <plugin>gz_ros2_control/GazeboSimSystem</plugin>
-      </xacro:if>
-      <xacro:unless value="${sim}">
-        <plugin>fairino_hardware/FairinoHardwareInterface</plugin>
-        <param name="robot_ip">$(arg robot_ip)</param>
-      </xacro:unless>
+      <plugin>fairino_hardware/FairinoHardwareInterface</plugin>
+      <param name="robot_ip">$(arg robot_ip)</param>
     </hardware>
     <xacro:macro name="controlled_joint" params="name">
@@ -80,8 +73,4 @@
           <param name="initial_value">${initial_positions[name]}</param>
         </state_interface>
-        <xacro:if value="${sim}">
-          <state_interface name="velocity"/>
-          <state_interface name="effort"/>
-        </xacro:if>
       </joint>
     </xacro:macro>
@@ -93,11 +82,3 @@
     <xacro:controlled_joint name="joint6"/>
   </ros2_control>
-  <xacro:if value="${sim}">
-    <gazebo>
-      <plugin filename="gz_ros2_control-system"
-        name="gz_ros2_control::GazeboSimROS2ControlPlugin">
-        <parameters>$(arg ros2_controllers_file)</parameters>
-      </plugin>
-    </gazebo>
-  </xacro:if>
 </robot>

File: src/dracoviloc_description/urdf/fairino3_v6_macro.xacro (robot description, xacro)
@@ -1,5 +1,5 @@
 <?xml version="1.0"?>
 <robot xmlns:xacro="http://www.ros.org/wiki/xacro">
-  <xacro:macro name="fairino3_v6_robot_prefixed" params="prefix sim:=false">
+  <xacro:macro name="fairino3_v6_robot_prefixed" params="prefix">
   <link
     name="${prefix}base_link">
@@ -42,10 +42,4 @@
     </collision>
   </link>
-  <xacro:if value="${sim}">
-    <gazebo reference="${prefix}base_link">
-      <static>true</static>
-      <self_collide>true</self_collide>
-    </gazebo>
-  </xacro:if>
   <link
     name="${prefix}shoulder_link">
@@ -88,9 +82,4 @@
     </collision>
   </link>
-  <xacro:if value="${sim}">
-    <gazebo reference="${prefix}shoulder_link">
-      <self_collide>true</self_collide>
-    </gazebo>
-  </xacro:if>
   <joint
     name="${prefix}joint1"
@@ -105,51 +94,21 @@
     <axis
       xyz="0 0 1" />
-    <xacro:unless value="${sim}">
-      <limit
+    <limit
         lower="-3.0543"
         upper="3.0543"
         effort="150"
         velocity="3.15" />
-    </xacro:unless>
-    <xacro:if value="${sim}">
-      <limit
-        lower="-3.0543"
-        upper="3.0543"
-        effort="150"
-        velocity="3.15" />
-    </xacro:if>
-    <calibration
-      rising="0"
-      falling="0" />
-    <dynamics
-      damping="0"
-      friction="0" />
-    <xacro:unless value="${sim}">
-      <safety_controller
+    <calibration
+      rising="0"
+      falling="0" />
+    <dynamics
+      damping="0"
+      friction="0" />
+    <safety_controller
         soft_lower_limit="-3.0543"
         soft_upper_limit="3.0543"
         k_position="15"
         k_velocity="10" />
-    </xacro:unless>
-    <xacro:if value="${sim}">
-      <safety_controller
-        soft_lower_limit="-3.0543"
-        soft_upper_limit="3.0543"
-        k_position="15"
-        k_velocity="10" />
-    </xacro:if>
-  </joint>
-  <xacro:if value="${sim}">
-    <transmission name="${prefix}joint1_trans">
-      <type>transmission_interface/SimpleTransmission</type>
-      <joint name="${prefix}joint1">
-        <hardwareInterface>hardware_interface/PositionJointInterface</hardwareInterface>
-      </joint>
-      <actuator name="${prefix}joint1_motor">
-        <hardwareInterface>hardware_interface/PositionJointInterface</hardwareInterface>
-        <mechanicalReduction>1</mechanicalReduction>
-      </actuator>
-    </transmission>
-  </xacro:if>
+  </joint>
   <link
     name="${prefix}upperarm_link">
@@ -192,9 +151,4 @@
     </collision>
   </link>
-  <xacro:if value="${sim}">
-    <gazebo reference="${prefix}upperarm_link">
-      <self_collide>true</self_collide>
-    </gazebo>
-  </xacro:if>
   <joint
     name="${prefix}joint2"
@@ -209,51 +163,21 @@
     <axis
       xyz="0 0 1" />
-    <xacro:unless value="${sim}">
-      <limit
+    <limit
         lower="-4.6251"
         upper="1.4835"
         effort="150"
         velocity="3.15" />
-    </xacro:unless>
-    <xacro:if value="${sim}">
-      <limit
-        lower="-4.6251"
-        upper="1.4835"
-        effort="150"
-        velocity="3.15" />
-    </xacro:if>
-    <calibration
-      rising="0"
-      falling="0" />
-    <dynamics
-      damping="0"
-      friction="0" />
-    <xacro:unless value="${sim}">
-      <safety_controller
+    <calibration
+      rising="0"
+      falling="0" />
+    <dynamics
+      damping="0"
+      friction="0" />
+    <safety_controller
         soft_lower_limit="-4.6251"
         soft_upper_limit="1.4835"
         k_position="15"
         k_velocity="10" />
-    </xacro:unless>
-    <xacro:if value="${sim}">
-      <safety_controller
-        soft_lower_limit="-4.6251"
-        soft_upper_limit="1.4835"
-        k_position="15"
-        k_velocity="10" />
-    </xacro:if>
-  </joint>
-  <xacro:if value="${sim}">
-    <transmission name="${prefix}joint2_trans">
-      <type>transmission_interface/SimpleTransmission</type>
-      <joint name="${prefix}joint2">
-        <hardwareInterface>hardware_interface/PositionJointInterface</hardwareInterface>
-      </joint>
-      <actuator name="${prefix}joint2_motor">
-        <hardwareInterface>hardware_interface/PositionJointInterface</hardwareInterface>
-        <mechanicalReduction>1</mechanicalReduction>
-      </actuator>
-    </transmission>
-  </xacro:if>
+  </joint>
   <link
     name="${prefix}forearm_link">
@@ -296,9 +220,4 @@
     </collision>
   </link>
-  <xacro:if value="${sim}">
-    <gazebo reference="${prefix}forearm_link">
-      <self_collide>true</self_collide>
-    </gazebo>
-  </xacro:if>
   <joint
     name="${prefix}joint3"
@@ -313,51 +232,21 @@
     <axis
       xyz="0 0 1" />
-    <xacro:unless value="${sim}">
-      <limit
+    <limit
         lower="-2.8274"
         upper="2.8274"
         effort="150"
         velocity="3.15" />
-    </xacro:unless>
-    <xacro:if value="${sim}">
-      <limit
-        lower="-2.8274"
-        upper="2.8274"
-        effort="150"
-        velocity="3.15" />
-    </xacro:if>
-    <calibration
-      rising="0"
-      falling="0" />
-    <dynamics
-      damping="0"
-      friction="0" />
-    <xacro:unless value="${sim}">
-      <safety_controller
+    <calibration
+      rising="0"
+      falling="0" />
+    <dynamics
+      damping="0"
+      friction="0" />
+    <safety_controller
         soft_lower_limit="-2.8274"
         soft_upper_limit="2.8274"
         k_position="15"
         k_velocity="10" />
-    </xacro:unless>
-    <xacro:if value="${sim}">
-      <safety_controller
-        soft_lower_limit="-2.8274"
-        soft_upper_limit="2.8274"
-        k_position="15"
-        k_velocity="10" />
-    </xacro:if>
-  </joint>
-  <xacro:if value="${sim}">
-    <transmission name="${prefix}joint3_trans">
-      <type>transmission_interface/SimpleTransmission</type>
-      <joint name="${prefix}joint3">
-        <hardwareInterface>hardware_interface/PositionJointInterface</hardwareInterface>
-      </joint>
-      <actuator name="${prefix}joint3_motor">
-        <hardwareInterface>hardware_interface/PositionJointInterface</hardwareInterface>
-        <mechanicalReduction>1</mechanicalReduction>
-      </actuator>
-    </transmission>
-  </xacro:if>
+  </joint>
   <link
     name="${prefix}wrist1_link">
@@ -400,9 +289,4 @@
     </collision>
   </link>
-  <xacro:if value="${sim}">
-    <gazebo reference="${prefix}wrist1_link">
-      <self_collide>true</self_collide>
-    </gazebo>
-  </xacro:if>
   <joint
     name="${prefix}joint4"
@@ -417,51 +301,21 @@
     <axis
       xyz="0 0 1" />
-    <xacro:unless value="${sim}">
-      <limit
+    <limit
         lower="-6.28319"
         upper="6.28319"
         effort="28"
         velocity="3.2" />
-    </xacro:unless>
-    <xacro:if value="${sim}">
-      <limit
-        lower="-6.28319"
-        upper="6.28319"
-        effort="28"
-        velocity="3.2" />
-    </xacro:if>
-    <calibration
-      rising="0"
-      falling="0" />
-    <dynamics
-      damping="0"
-      friction="0" />
-    <xacro:unless value="${sim}">
-      <safety_controller
+    <calibration
+      rising="0"
+      falling="0" />
+    <dynamics
+      damping="0"
+      friction="0" />
+    <safety_controller
         soft_lower_limit="-6.28319"
         soft_upper_limit="6.28319"
         k_position="15"
         k_velocity="10" />
-    </xacro:unless>
-    <xacro:if value="${sim}">
-      <safety_controller
-        soft_lower_limit="-6.28319"
-        soft_upper_limit="6.28319"
-        k_position="15"
-        k_velocity="10" />
-    </xacro:if>
-  </joint>
-  <xacro:if value="${sim}">
-    <transmission name="${prefix}joint4_trans">
-      <type>transmission_interface/SimpleTransmission</type>
-      <joint name="${prefix}joint4">
-        <hardwareInterface>hardware_interface/PositionJointInterface</hardwareInterface>
-      </joint>
-      <actuator name="${prefix}joint4_motor">
-        <hardwareInterface>hardware_interface/PositionJointInterface</hardwareInterface>
-        <mechanicalReduction>1</mechanicalReduction>
-      </actuator>
-    </transmission>
-  </xacro:if>
+  </joint>
   <link
     name="${prefix}wrist2_link">
@@ -504,9 +358,4 @@
     </collision>
   </link>
-  <xacro:if value="${sim}">
-    <gazebo reference="${prefix}wrist2_link">
-      <self_collide>true</self_collide>
-    </gazebo>
-  </xacro:if>
   <joint
     name="${prefix}joint5"
@@ -521,51 +370,21 @@
     <axis
       xyz="0 0 1" />
-    <xacro:unless value="${sim}">
-      <limit
+    <limit
         lower="-6.28319"
         upper="6.28319"
         effort="28"
         velocity="3.2" />
-    </xacro:unless>
-    <xacro:if value="${sim}">
-      <limit
-        lower="-6.28319"
-        upper="6.28319"
-        effort="28"
-        velocity="3.2" />
-    </xacro:if>
-    <calibration
-      rising="0"
-      falling="0" />
-    <dynamics
-      damping="0"
-      friction="0" />
-    <xacro:unless value="${sim}">
-      <safety_controller
+    <calibration
+      rising="0"
+      falling="0" />
+    <dynamics
+      damping="0"
+      friction="0" />
+    <safety_controller
         soft_lower_limit="-6.28319"
         soft_upper_limit="6.28319"
         k_position="15"
         k_velocity="10" />
-    </xacro:unless>
-    <xacro:if value="${sim}">
-      <safety_controller
-        soft_lower_limit="-6.28319"
-        soft_upper_limit="6.28319"
-        k_position="15"
-        k_velocity="10" />
-    </xacro:if>
-  </joint>
-  <xacro:if value="${sim}">
-    <transmission name="${prefix}joint5_trans">
-      <type>transmission_interface/SimpleTransmission</type>
-      <joint name="${prefix}joint5">
-        <hardwareInterface>hardware_interface/PositionJointInterface</hardwareInterface>
-      </joint>
-      <actuator name="${prefix}joint5_motor">
-        <hardwareInterface>hardware_interface/PositionJointInterface</hardwareInterface>
-        <mechanicalReduction>1</mechanicalReduction>
-      </actuator>
-    </transmission>
-  </xacro:if>
+  </joint>
   <link
     name="${prefix}wrist3_link">
@@ -608,9 +427,4 @@
     </collision>
   </link>
-  <xacro:if value="${sim}">
-    <gazebo reference="${prefix}wrist3_link">
-      <self_collide>true</self_collide>
-    </gazebo>
-  </xacro:if>
   <joint
     name="${prefix}joint6"
@@ -625,51 +439,21 @@
     <axis
       xyz="0 0 1" />
-    <xacro:unless value="${sim}">
-      <limit
+    <limit
         lower="-6.28319"
         upper="6.28319"
         effort="28"
         velocity="3.2" />
-    </xacro:unless>
-    <xacro:if value="${sim}">
-      <limit
-        lower="-6.28319"
-        upper="6.28319"
-        effort="28"
-        velocity="3.2" />
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
Commit message: removed gazebo entirely

File: src/dracoviloc_description/urdf/dracoviloc.urdf.xacro (robot description, xacro)
@@ -2,4 +2,5 @@
 <robot xmlns:xacro="http://www.ros.org/wiki/xacro" name="dracoviloc">
   <xacro:arg name="robot_ip" default="192.168.58.2"/>
+  <xacro:arg name="hardware_mode" default="mock"/>
   <xacro:arg name="initial_positions_file"
     default="$(find dracoviloc_description)/config/initial_positions.yaml"/>
@@ -8,4 +9,5 @@
   <xacro:property name="initial_positions"
     value="${xacro.load_yaml('$(arg initial_positions_file)')['initial_positions']}"/>
+  <xacro:property name="hardware_mode" value="$(arg hardware_mode)"/>
   <xacro:include filename="$(find dracoviloc_description)/urdf/fairino3_v6_macro.xacro"/>
   <link name="world"/>
@@ -64,6 +66,11 @@
   <ros2_control name="fairino_arm_system" type="system">
     <hardware>
-      <plugin>fairino_hardware/FairinoHardwareInterface</plugin>
-      <param name="robot_ip">$(arg robot_ip)</param>
+      <xacro:if value="${hardware_mode == 'mock'}">
+        <plugin>mock_components/GenericSystem</plugin>
+      </xacro:if>
+      <xacro:if value="${hardware_mode == 'real'}">
+        <plugin>fairino_hardware/FairinoHardwareInterface</plugin>
+        <param name="robot_ip">$(arg robot_ip)</param>
+      </xacro:if>
     </hardware>
     <xacro:macro name="controlled_joint" params="name">
