Commit message: feat(dual_arm): add dual-arm co-tracking and parallel gaze alignment

File: src/dracoviloc_description/urdf/dracoviloc.urdf.xacro (robot description, xacro)
@@ -1,5 +1,11 @@
 <?xml version="1.0"?>
 <robot xmlns:xacro="http://www.ros.org/wiki/xacro" name="dracoviloc">
+  <xacro:arg name="dual_arm" default="false"/>
   <xacro:arg name="robot_ip" default="192.168.58.2"/>
+  <xacro:arg name="left_robot_ip" default="192.168.58.2"/>
+  <xacro:arg name="right_robot_ip" default="192.168.58.3"/>
+  <xacro:arg name="second_arm_x" default="-0.75"/>
+  <xacro:arg name="second_arm_y" default="0.0"/>
+  <xacro:arg name="second_arm_z" default="0.0"/>
   <xacro:arg name="hardware_mode" default="mock"/>
   <xacro:arg name="initial_positions_file"
@@ -10,82 +16,191 @@
     value="${xacro.load_yaml('$(arg initial_positions_file)')['initial_positions']}"/>
   <xacro:property name="hardware_mode" value="$(arg hardware_mode)"/>
+  <xacro:property name="is_dual_arm" value="$(arg dual_arm)"/>
   <xacro:include filename="$(find dracoviloc_description)/urdf/fairino3_v6_macro.xacro"/>
   <link name="world"/>
-  <joint name="world_to_base" type="fixed">
-    <parent link="world"/>
-    <child link="base_link"/>
-  </joint>
-  <xacro:fairino3_v6_robot_prefixed prefix=""/>
-  <!-- D435i body convention inherited from Vicoman:
-       +X forward/view direction, +Y left, +Z up.
-       Adjust these three properties to calibrate the wrist-to-camera mount. -->
+  <!-- Mount offsets for sensors on wrist3 -->
   <xacro:property name="d435i_mount_x" value="0.0"/>
   <xacro:property name="d435i_mount_y" value="0.0"/>
   <xacro:property name="d435i_mount_z" value="0.1"/>
-  <link name="d435i_link">
-    <visual>
-      <geometry><box size="0.025 0.09 0.025"/></geometry>
-      <material name="camera_grey"><color rgba="0.25 0.25 0.25 1.0"/></material>
-    </visual>
-    <collision><geometry><box size="0.025 0.09 0.025"/></geometry></collision>
-    <inertial>
-      <mass value="0.1"/>
-      <inertia ixx="0.000073" ixy="0" ixz="0"
-               iyy="0.000010" iyz="0" izz="0.000073"/>
-    </inertial>
-  </link>
-  <joint name="wrist3_to_d435i" type="fixed">
-    <parent link="wrist3_link"/>
-    <child link="d435i_link"/>
-    <origin xyz="${d435i_mount_x} ${d435i_mount_y} ${d435i_mount_z}"
-            rpy="0 0 0"/>
-  </joint>
-  <!-- UMA16v2 microphone-array frame. ODAS directions are expressed in this
-       frame; +Z is normal to the microphone plane. These placeholder mount
-       dimensions must be replaced with measurements from the final bracket. -->
   <xacro:property name="odas_mount_x" value="0.0"/>
   <xacro:property name="odas_mount_y" value="0.0"/>
   <xacro:property name="odas_mount_z" value="0.13"/>
-  <link name="odas_link">
-    <visual>
-      <geometry><box size="0.126 0.126 0.008"/></geometry>
-      <material name="odas_blue"><color rgba="0.05 0.25 0.8 0.8"/></material>
-    </visual>
-    <collision><geometry><box size="0.126 0.126 0.008"/></geometry></collision>
-    <inertial>
-      <mass value="0.08"/>
-      <inertia ixx="0.000106" ixy="0" ixz="0"
-               iyy="0.000106" iyz="0" izz="0.000212"/>
-    </inertial>
-  </link>
-  <joint name="wrist3_to_odas" type="fixed">
-    <parent link="wrist3_link"/>
-    <child link="odas_link"/>
-    <origin xyz="${odas_mount_x} ${odas_mount_y} ${odas_mount_z}" rpy="0 0 0"/>
-  </joint>
-  <ros2_control name="fairino_arm_system" type="system">
-    <hardware>
-      <xacro:if value="${hardware_mode == 'mock'}">
-        <plugin>mock_components/GenericSystem</plugin>
-      </xacro:if>
-      <xacro:if value="${hardware_mode == 'real'}">
-        <plugin>fairino_hardware/FairinoHardwareInterface</plugin>
-        <param name="robot_ip">$(arg robot_ip)</param>
-      </xacro:if>
-    </hardware>
-    <xacro:macro name="controlled_joint" params="name">
-      <joint name="${name}">
-        <command_interface name="position"/>
-        <state_interface name="position">
-          <param name="initial_value">${initial_positions[name]}</param>
-        </state_interface>
-      </joint>
-    </xacro:macro>
-    <xacro:controlled_joint name="joint1"/>
-    <xacro:controlled_joint name="joint2"/>
-    <xacro:controlled_joint name="joint3"/>
-    <xacro:controlled_joint name="joint4"/>
-    <xacro:controlled_joint name="joint5"/>
-    <xacro:controlled_joint name="joint6"/>
-  </ros2_control>
+  <!-- ================= SINGLE ARM MODE ================= -->
+  <xacro:unless value="${is_dual_arm}">
+    <joint name="world_to_base" type="fixed">
+      <parent link="world"/>
+      <child link="base_link"/>
+    </joint>
+    <xacro:fairino3_v6_robot_prefixed prefix=""/>
+    <link name="d435i_link">
+      <visual>
+        <geometry><box size="0.025 0.09 0.025"/></geometry>
+        <material name="camera_grey"><color rgba="0.25 0.25 0.25 1.0"/></material>
+      </visual>
+      <collision><geometry><box size="0.025 0.09 0.025"/></geometry></collision>
+      <inertial>
+        <mass value="0.1"/>
+        <inertia ixx="0.000073" ixy="0" ixz="0"
+                 iyy="0.000010" iyz="0" izz="0.000073"/>
+      </inertial>
+    </link>
+    <joint name="wrist3_to_d435i" type="fixed">
+      <parent link="wrist3_link"/>
+      <child link="d435i_link"/>
+      <origin xyz="${d435i_mount_x} ${d435i_mount_y} ${d435i_mount_z}" rpy="0 0 0"/>
+    </joint>
+    <link name="odas_link">
+      <visual>
+        <geometry><box size="0.126 0.126 0.008"/></geometry>
+        <material name="odas_blue"><color rgba="0.05 0.25 0.8 0.8"/></material>
+      </visual>
+      <collision><geometry><box size="0.126 0.126 0.008"/></geometry></collision>
+      <inertial>
+        <mass value="0.08"/>
+        <inertia ixx="0.000106" ixy="0" ixz="0"
+                 iyy="0.000106" iyz="0" izz="0.000212"/>
+      </inertial>
+    </link>
+    <joint name="wrist3_to_odas" type="fixed">
+      <parent link="wrist3_link"/>
+      <child link="odas_link"/>
+      <origin xyz="${odas_mount_x} ${odas_mount_y} ${odas_mount_z}" rpy="0 0 0"/>
+    </joint>
+    <ros2_control name="fairino_arm_system" type="system">
+      <hardware>
+        <xacro:if value="${hardware_mode == 'mock'}">
+          <plugin>mock_components/GenericSystem</plugin>
+        </xacro:if>
+        <xacro:if value="${hardware_mode == 'real'}">
+          <plugin>fairino_hardware/FairinoHardwareInterface</plugin>
+          <param name="robot_ip">$(arg robot_ip)</param>
+        </xacro:if>
+      </hardware>
+      <xacro:macro name="controlled_joint" params="name">
+        <joint name="${name}">
+          <command_interface name="position"/>
+          <state_interface name="position">
+            <param name="initial_value">${initial_positions[name]}</param>
+          </state_interface>
+        </joint>
+      </xacro:macro>
+      <xacro:controlled_joint name="joint1"/>
+      <xacro:controlled_joint name="joint2"/>
+      <xacro:controlled_joint name="joint3"/>
+      <xacro:controlled_joint name="joint4"/>
+      <xacro:controlled_joint name="joint5"/>
+      <xacro:controlled_joint name="joint6"/>
+    </ros2_control>
+  </xacro:unless>
+  <!-- ================= DUAL ARM MODE ================= -->
+  <xacro:if value="${is_dual_arm}">
+    <!-- Arm 1 (Left / Primary) base link at origin -->
+    <joint name="world_to_left_base" type="fixed">
+      <parent link="world"/>
+      <child link="left_base_link"/>
+      <origin xyz="0 0 0" rpy="0 0 0"/>
+    </joint>
+    <!-- Legacy base_link alias pointing to left_base_link -->
+    <link name="base_link"/>
+    <joint name="left_base_to_base_link" type="fixed">
+      <parent link="left_base_link"/>
+      <child link="base_link"/>
+      <origin xyz="0 0 0" rpy="0 0 0"/>
+    </joint>
+    <xacro:fairino3_v6_robot_prefixed prefix="left_"/>
+    <!-- Primary arm mounts sensors (D435i camera + ODAS microphone array) -->
+    <link name="d435i_link">
+      <visual>
+        <geometry><box size="0.025 0.09 0.025"/></geometry>
+        <material name="camera_grey"><color rgba="0.25 0.25 0.25 1.0"/></material>
+      </visual>
+      <collision><geometry><box size="0.025 0.09 0.025"/></geometry></collision>
+      <inertial>
+        <mass value="0.1"/>
+        <inertia ixx="0.000073" ixy="0" ixz="0"
+                 iyy="0.000010" iyz="0" izz="0.000073"/>
+      </inertial>
+    </link>
+    <joint name="left_wrist3_to_d435i" type="fixed">
+      <parent link="left_wrist3_link"/>
+      <child link="d435i_link"/>
+      <origin xyz="${d435i_mount_x} ${d435i_mount_y} ${d435i_mount_z}" rpy="0 0 0"/>
+    </joint>
+    <link name="odas_link">
+      <visual>
+        <geometry><box size="0.126 0.126 0.008"/></geometry>
+        <material name="odas_blue"><color rgba="0.05 0.25 0.8 0.8"/></material>
+      </visual>
+      <collision><geometry><box size="0.126 0.126 0.008"/></geometry></collision>
+      <inertial>
+        <mass value="0.08"/>
+        <inertia ixx="0.000106" ixy="0" ixz="0"
+                 iyy="0.000106" iyz="0" izz="0.000212"/>
+      </inertial>
+    </link>
+    <joint name="left_wrist3_to_odas" type="fixed">
+      <parent link="left_wrist3_link"/>
+      <child link="odas_link"/>
+      <origin xyz="${odas_mount_x} ${odas_mount_y} ${odas_mount_z}" rpy="0 0 0"/>
+    </joint>
+    <!-- Arm 2 (Right / Follower) base link at 75cm offset along -X (to the left of master arm) -->
+    <joint name="world_to_right_base" type="fixed">
+      <parent link="world"/>
+      <child link="right_base_link"/>
+      <origin xyz="$(arg second_arm_x) $(arg second_arm_y) $(arg second_arm_z)" rpy="0 0 0"/>
+    </joint>
+    <xacro:fairino3_v6_robot_prefixed prefix="right_"/>
+    <!-- Follower arm end-effector tool / optical pointer link -->
+    <link name="right_tool_link">
+      <visual>
+        <geometry><cylinder radius="0.04" length="0.03"/></geometry>
+        <material name="right_tool_cyan"><color rgba="0.1 0.7 0.8 1.0"/></material>
+      </visual>
+      <collision><geometry><cylinder radius="0.04" length="0.03"/></geometry></collision>
+      <inertial>
+        <mass value="0.05"/>
+        <inertia ixx="0.00003" ixy="0" ixz="0"
+                 iyy="0.00003" iyz="0" izz="0.00004"/>
+      </inertial>
+    </link>
+    <joint name="right_wrist3_to_tool" type="fixed">
+      <parent link="right_wrist3_link"/>
+      <child link="right_tool_link"/>
+      <origin xyz="0 0 0.05" rpy="0 0 0"/>
+    </joint>
+    <ros2_control name="fairino_dual_arm_system" type="system">
+      <hardware>
+        <xacro:if value="${hardware_mode == 'mock'}">
+          <plugin>mock_components/GenericSystem</plugin>
+        </xacro:if>
+        <xacro:if value="${hardware_mode == 'real'}">
+          <plugin>fairino_hardware/FairinoHardwareInterface</plugin>
+          <param name="left_robot_ip">$(arg left_robot_ip)</param>
+          <param name="right_robot_ip">$(arg right_robot_ip)</param>
+        </xacro:if>
+      </hardware>
+      <xacro:macro name="dual_controlled_joint" params="name">
+        <joint name="${name}">
+          <command_interface name="position"/>
+          <state_interface name="position">
+            <param name="initial_value">${initial_positions[name]}</param>
+          </state_interface>
+        </joint>
+      </xacro:macro>
+      <!-- Left arm joints -->
+      <xacro:dual_controlled_joint name="left_joint1"/>
+      <xacro:dual_controlled_joint name="left_joint2"/>
+      <xacro:dual_controlled_joint name="left_joint3"/>
+      <xacro:dual_controlled_joint name="left_joint4"/>
+      <xacro:dual_controlled_joint name="left_joint5"/>
+      <xacro:dual_controlled_joint name="left_joint6"/>
+      <!-- Right arm joints -->
+      <xacro:dual_controlled_joint name="right_joint1"/>
+      <xacro:dual_controlled_joint name="right_joint2"/>
+      <xacro:dual_controlled_joint name="right_joint3"/>
+      <xacro:dual_controlled_joint name="right_joint4"/>
+      <xacro:dual_controlled_joint name="right_joint5"/>
+      <xacro:dual_controlled_joint name="right_joint6"/>
+    </ros2_control>
+  </xacro:if>
 </robot>

Commit message: worked on improving the GUI

File: src/dracoviloc_description/urdf/dracoviloc.urdf.xacro (robot description, xacro)
@@ -20,7 +20,7 @@
   <link name="world"/>
   <!-- Mount offsets for sensors on wrist3 -->
-  <xacro:property name="d435i_mount_x" value="0.0"/>
-  <xacro:property name="d435i_mount_y" value="0.0"/>
-  <xacro:property name="d435i_mount_z" value="0.1"/>
+  <xacro:property name="micarray_camera_mount_x" value="0.0"/>
+  <xacro:property name="micarray_camera_mount_y" value="0.0"/>
+  <xacro:property name="micarray_camera_mount_z" value="0.1"/>
   <xacro:property name="odas_mount_x" value="0.0"/>
   <xacro:property name="odas_mount_y" value="0.0"/>
@@ -33,5 +33,5 @@
     </joint>
     <xacro:fairino3_v6_robot_prefixed prefix=""/>
-    <link name="d435i_link">
+    <link name="micarray_camera_link">
       <visual>
         <geometry><box size="0.025 0.09 0.025"/></geometry>
@@ -45,8 +45,8 @@
       </inertial>
     </link>
-    <joint name="wrist3_to_d435i" type="fixed">
+    <joint name="wrist3_to_micarray_camera" type="fixed">
       <parent link="wrist3_link"/>
-      <child link="d435i_link"/>
-      <origin xyz="${d435i_mount_x} ${d435i_mount_y} ${d435i_mount_z}" rpy="0 0 0"/>
+      <child link="micarray_camera_link"/>
+      <origin xyz="${micarray_camera_mount_x} ${micarray_camera_mount_y} ${micarray_camera_mount_z}" rpy="0 0 0"/>
     </joint>
     <link name="odas_link">
@@ -109,6 +109,6 @@
     </joint>
     <xacro:fairino3_v6_robot_prefixed prefix="left_"/>
-    <!-- Primary arm mounts sensors (D435i camera + ODAS microphone array) -->
-    <link name="d435i_link">
+    <!-- Primary arm mounts sensors (mic-array camera + ODAS microphone array) -->
+    <link name="micarray_camera_link">
       <visual>
         <geometry><box size="0.025 0.09 0.025"/></geometry>
@@ -122,8 +122,8 @@
       </inertial>
     </link>
-    <joint name="left_wrist3_to_d435i" type="fixed">
+    <joint name="left_wrist3_to_micarray_camera" type="fixed">
       <parent link="left_wrist3_link"/>
-      <child link="d435i_link"/>
-      <origin xyz="${d435i_mount_x} ${d435i_mount_y} ${d435i_mount_z}" rpy="0 0 0"/>
+      <child link="micarray_camera_link"/>
+      <origin xyz="${micarray_camera_mount_x} ${micarray_camera_mount_y} ${micarray_camera_mount_z}" rpy="0 0 0"/>
     </joint>
     <link name="odas_link">

Commit message: Stabilize cobot tracking and update GUI pipelines

File: src/dracoviloc_description/urdf/dracoviloc.urdf.xacro (robot description, xacro)
@@ -50,4 +50,12 @@
       <origin xyz="${micarray_camera_mount_x} ${micarray_camera_mount_y} ${micarray_camera_mount_z}" rpy="0 0 0"/>
     </joint>
+    <!-- At the home pose this matches the former table_mic_link axes, but
+         follows the wrist when the camera and microphone array move. -->
+    <link name="micarray_direction_link"/>
+    <joint name="micarray_camera_to_direction" type="fixed">
+      <parent link="micarray_camera_link"/>
+      <child link="micarray_direction_link"/>
+      <origin xyz="0 0 0" rpy="0 0 3.141592653589793"/>
+    </joint>
     <link name="odas_link">
       <visual>
@@ -126,4 +134,10 @@
       <child link="micarray_camera_link"/>
       <origin xyz="${micarray_camera_mount_x} ${micarray_camera_mount_y} ${micarray_camera_mount_z}" rpy="0 0 0"/>
+    </joint>
+    <link name="micarray_direction_link"/>
+    <joint name="micarray_camera_to_direction" type="fixed">
+      <parent link="micarray_camera_link"/>
+      <child link="micarray_direction_link"/>
+      <origin xyz="0 0 0" rpy="0 0 3.141592653589793"/>
     </joint>
     <link name="odas_link">
